File: Reloj_V1/Reloj_V1.kicad_pcb (KiCad board)
At the start: 2 copper layers, 231.3 x 123.5 mm, 48 parts, among them J1 Barrel_Jack_MountingPin, J2 Screw_Terminal_01x02, U11 74HC595, U12 ULN2803A, U13 74HC595, U14 ULN2803A, U15 74HC595, U16 ULN2803A, U17 74HC595, U18 ULN2803A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

Commit message: .
Routing:
- net RCLK_4: track 167.9 -> 170.6 mm
- net +5V: track 192.4 -> 191.2 mm
